File: schematic/schematic.kicad_pcb (KiCad board)
At the start: 2 copper layers, 11 parts, among them Q1 IRLZ34N, SW1 MODE, SW2 UP, SW3 DOWN, SW4 SW_Push, U1 TM1637Display

Commit message: draw schematics
Parts:
- added R1: R, Resistor_THT:R_Axial_DIN0204_L3.6mm_D1.6mm_P5.08mm_Vertical, F.Cu at (3.81, 77.5)
- added R2: R, Resistor_THT:R_Axial_DIN0204_L3.6mm_D1.6mm_P5.08mm_Vertical, F.Cu at (103.0, 91.8)
- added R3: R, Resistor_THT:R_Axial_DIN0204_L3.6mm_D1.6mm_P5.08mm_Vertical, F.Cu at (171.4, 130.8)
- added R4: R, Resistor_THT:R_Axial_DIN0204_L3.6mm_D1.6mm_P5.08mm_Vertical, F.Cu at (-0.64, 47.3)
- added R5: R, Resistor_THT:R_Axial_DIN0204_L3.6mm_D1.6mm_P5.08mm_Vertical, F.Cu at (155.2, 46.8)
- SW1: value MODE -> UP
- SW2: value UP -> DOWN
- SW3: value DOWN -> CONFIRM
- SW4: value SW_Push -> MODE
- moved D3 417.4 mm to (-22.5, 69.3)
- moved D1 337.3 mm to (115.8, 80.7)
- moved A1 297.9 mm to (66.8, 22.6)
- moved D2 288.8 mm to (128.8, 72.2)
- moved Q1 288.8 mm to (145.3, 49.1)
- moved SW1 288.8 mm to (108.0, 71.4)
- moved SW4 288.8 mm to (118.6, 71.4)
- moved U1 288.8 mm to (103.7, 71.7)
- moved SW2 288.8 mm to (103.4, 83.7)
- moved SW3 288.8 mm to (144.1, 53.2)
- moved RTC1 215.4 mm to (168.9, 14.0), turned to 270 degrees
Connections:
- net Net-(Q1-Pad2) renamed lamp_gnd
- A1 pad 10: Net-(A1-Pad10) -> switch_mode
- A1 pad 11: Net-(A1-Pad11) -> display_dio
- A1 pad 12: Net-(A1-Pad12) -> display_clk
- A1 pad 20: Net-(A1-Pad20) -> switch_confirm
- A1 pad 29: Net-(A1-Pad29) -> display_gnd
- A1 pad 30: Net-(A1-Pad30) -> display_vcc
- A1 pad 4: Net-(A1-Pad4) -> display_gnd
- A1 pad 5: Net-(A1-Pad5) -> led_off
- A1 pad 6: Net-(A1-Pad6) -> led_on
- A1 pad 7: Net-(A1-Pad7) -> led_time
- A1 pad 8: Net-(A1-Pad8) -> switch_down
- A1 pad 9: Net-(A1-Pad9) -> switch_up
- D1 pad 2: Net-(D1-Pad2) -> led_off
- D2 pad 2: Net-(D2-Pad2) -> led_on
- D3 pad 2: Net-(D3-Pad2) -> led_time
- Q1 pad 3: Net-(Q1-Pad3) -> display_gnd
- RTC1 pad 1: Net-(RTC1-Pad1) -> display_gnd
- RTC1 pad 2: Net-(RTC1-Pad2) -> display_vcc
- RTC1 pad 3: Net-(RTC1-Pad3) -> Net-(A1-Pad23)
- RTC1 pad 4: Net-(RTC1-Pad4) -> Net-(A1-Pad24)
- SW1 pad 1: Net-(SW1-Pad1) -> display_gnd
- SW1 pad 2: Net-(A1-Pad10) -> switch_up
- SW2 pad 1: Net-(SW2-Pad1) -> display_gnd
- SW2 pad 2: Net-(A1-Pad9) -> switch_down
- SW3 pad 1: Net-(SW3-Pad1) -> display_gnd
- SW3 pad 2: Net-(A1-Pad8) -> switch_confirm
- SW4 pad 1: Net-(SW4-Pad1) -> display_gnd
- SW4 pad 2: Net-(SW4-Pad2) -> switch_mode
- U1 pad 1: Net-(U1-Pad1) -> display_clk
- U1 pad 2: Net-(U1-Pad2) -> display_dio
- U1 pad 3: Net-(U1-Pad3) -> display_gnd
- U1 pad 4: Net-(U1-Pad4) -> display_vcc

Commit message: update board
Parts:
- added J1: lamp VCC, Connector_Wire:SolderWirePad_1x01_Drill0.8mm, F.Cu at (-35.6, 30.5)
- added J10: button MODE, Connector_Wire:SolderWirePad_1x01_Drill0.8mm, F.Cu at (221.0, -17.8)
- added J11: button GND, Connector_Wire:SolderWirePad_1x01_Drill0.8mm, F.Cu at (205.7, -17.8)
- added J12: display DIO, Connector_Wire:SolderWirePad_1x01_Drill0.8mm, F.Cu at (139.7, -17.8)
- added J13: display CLK, Connector_Wire:SolderWirePad_1x01_Drill0.8mm, F.Cu at (134.6, -17.8)
- added J14: display VCC, Connector_Wire:SolderWirePad_1x01_Drill0.8mm, F.Cu at (190.5, -17.8)
- added J15: display GND, Connector_Wire:SolderWirePad_1x01_Drill0.8mm, F.Cu at (195.6, -17.8)
- added J16: led OFF, Connector_Wire:SolderWirePad_1x01_Drill0.8mm, F.Cu at (-12.7, 5.08)
- added J17: led ON, Connector_Wire:SolderWirePad_1x01_Drill0.8mm, F.Cu at (-12.7, -2.54)
- added J18: led TIME, Connector_Wire:SolderWirePad_1x01_Drill0.8mm, F.Cu at (-12.7, -10.2)
- added J19: led GND, Connector_Wire:SolderWirePad_1x01_Drill0.8mm, F.Cu at (-12.7, 10.2)
- added J2: lamp GND, Connector_Wire:SolderWirePad_1x01_Drill0.8mm, F.Cu at (-35.6, 38.1)
- added J20: button CONFIRM, Connector_Wire:SolderWirePad_1x01_Drill0.8mm, F.Cu at (5.08, 88.9)
- added J21: button DOWN, Connector_Wire:SolderWirePad_1x01_Drill0.8mm, F.Cu at (5.08, 68.6)
- added J22: button UP, Connector_Wire:SolderWirePad_1x01_Drill0.8mm, F.Cu at (5.08, 76.2)
- added J23: button MODE, Connector_Wire:SolderWirePad_1x01_Drill0.8mm, F.Cu at (5.08, 83.8)
- added J24: button GND, Connector_Wire:SolderWirePad_1x01_Drill0.8mm, F.Cu at (5.08, 96.5)
- added J25: display DIO, Connector_Wire:SolderWirePad_1x01_Drill0.8mm, F.Cu at (-10.2, 53.3)
- added J26: display CLK, Connector_Wire:SolderWirePad_1x01_Drill0.8mm, F.Cu at (-10.2, 58.4)
- added J27: display VCC, Connector_Wire:SolderWirePad_1x01_Drill0.8mm, F.Cu at (-10.2, 71.1)
- added J28: display GND, Connector_Wire:SolderWirePad_1x01_Drill0.8mm, F.Cu at (-10.2, 63.5)
- added J29: VCC, Connector_Wire:SolderWirePad_1x01_Drill0.8mm, F.Cu at (35.6, -5.08)
- added J3: led OFF, Connector_Wire:SolderWirePad_1x01_Drill0.8mm, F.Cu at (170.2, -17.8)
- added J30: VCC amp, Connector_Wire:SolderWirePad_1x01_Drill0.8mm, F.Cu at (12.7, -5.08)
- added J31: GND lamp, Connector_Wire:SolderWirePad_1x01_Drill0.8mm, F.Cu at (20.3, -5.08)
- added J32: GND, Connector_Wire:SolderWirePad_1x01_Drill0.8mm, F.Cu at (27.9, -5.08)
- added J4: led ON, Connector_Wire:SolderWirePad_1x01_Drill0.8mm, F.Cu at (175.3, -17.8)
- added J5: led TIME, Connector_Wire:SolderWirePad_1x01_Drill0.8mm, F.Cu at (180.3, -17.8)
- added J6: led GND, Connector_Wire:SolderWirePad_1x01_Drill0.8mm, F.Cu at (200.7, -17.8)
- added J7: button CONFIRM, Connector_Wire:SolderWirePad_1x01_Drill0.8mm, F.Cu at (236.2, -17.8)
- added J8: button DOWN, Connector_Wire:SolderWirePad_1x01_Drill0.8mm, F.Cu at (231.1, -17.8)
- added J9: button UP, Connector_Wire:SolderWirePad_1x01_Drill0.8mm, F.Cu at (226.1, -17.8)
- R1, R2, R3, R4, R5: footprint Resistor_THT:R_Axial_DIN0204_L3.6mm_D1.6mm_P5.08mm_Vertical -> Resistor_THT:R_Axial_DIN0207_L6.3mm_D2.5mm_P10.16mm_Horizontal
- SW1, SW2, SW3, SW4: footprint Button_Switch_THT:SW_PUSH_6mm_H5mm -> Button_Switch_THT:SW_PUSH-12mm
- moved D3 226.0 mm to (180.3, -30.5), turned to 270 degrees
- moved R4 206.4 mm to (190.5, -30.5)
- moved SW2 192.5 mm to (256.5, -33.0)
- moved R3 172.5 mm to (190.5, -40.6)
- moved SW1 167.3 mm to (238.8, -33.0)
- moved R2 167.3 mm to (190.5, -50.8)
- moved R5 164.2 mm to (-7.62, 25.4)
- moved SW3 156.2 mm to (274.3, -33.0)
- moved Q1 153.5 mm to (-7.62, 35.6)
- moved D1 146.5 mm to (180.3, -50.8), turned to 270 degrees
- moved SW4 146.3 mm to (221.0, -33.0)
- moved D2 124.0 mm to (180.3, -40.6), turned to 270 degrees
- moved RTC1 118.4 mm to (56.9, -24.4), turned to 0 degrees
- moved U1 117.3 mm to (144.8, -38.1)
- moved A1 37.8 mm to (29.2, 19.1)
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Connections:
- A1 pad 10: switch_mode -> Net-(A1-Pad10)
- A1 pad 11: display_dio -> Net-(A1-Pad11)
- A1 pad 12: display_clk -> Net-(A1-Pad12)
- A1 pad 20: switch_confirm -> Net-(A1-Pad20)
- A1 pad 29: display_gnd -> GND
- A1 pad 30: display_vcc -> +5V
- A1 pad 4: display_gnd -> GND
- A1 pad 5: led_off -> Net-(A1-Pad5)
- A1 pad 6: led_on -> Net-(A1-Pad6)
- A1 pad 7: led_time -> Net-(A1-Pad7)
- A1 pad 8: switch_down -> Net-(A1-Pad8)
- A1 pad 9: switch_up -> Net-(A1-Pad9)
- D1 pad 2: led_off -> Net-(D1-Pad2)
- D2 pad 2: led_on -> Net-(D2-Pad2)
- D3 pad 2: led_time -> Net-(D3-Pad2)
- Q1 pad 2: lamp_gnd -> Net-(J2-Pad1)
- Q1 pad 3: display_gnd -> Net-(J31-Pad1)
- R2 pad 2: display_gnd -> Net-(J6-Pad1)
- R3 pad 2: display_gnd -> Net-(J6-Pad1)
- R4 pad 2: display_gnd -> Net-(J6-Pad1)
- R5 pad 2: display_gnd -> GND
- RTC1 pad 1: display_gnd -> GND
- RTC1 pad 2: display_vcc -> +5V
- SW1 pad 1: display_gnd -> Net-(J11-Pad1)
- SW1 pad 2: switch_up -> Net-(J9-Pad1)
- SW2 pad 1: display_gnd -> Net-(J11-Pad1)
- SW2 pad 2: switch_down -> Net-(J8-Pad1)
- SW3 pad 1: display_gnd -> Net-(J11-Pad1)
- SW3 pad 2: switch_confirm -> Net-(J7-Pad1)
- SW4 pad 1: display_gnd -> Net-(J11-Pad1)
- SW4 pad 2: switch_mode -> Net-(J10-Pad1)
- U1 pad 1: display_clk -> Net-(J13-Pad1)
- U1 pad 2: display_dio -> Net-(J12-Pad1)
- U1 pad 3: display_gnd -> Net-(J15-Pad1)
- U1 pad 4: display_vcc -> Net-(J14-Pad1)
Routing:
- net Net-(J11-Pad1): track 0.00 -> 96.3 mm
- net Net-(J15-Pad1): track 0.00 -> 66.0 mm, vias 0 -> 2
- net Net-(J7-Pad1): track 0.00 -> 60.8 mm
- net Net-(J14-Pad1): track 0.00 -> 58.4 mm, vias 0 -> 2
- net Net-(J8-Pad1): track 0.00 -> 48.1 mm
- net Net-(D1-Pad2): track 0.00 -> 40.6 mm
- net Net-(J9-Pad1): track 0.00 -> 35.4 mm
- net Net-(J6-Pad1): track 0.00 -> 33.0 mm
- net Net-(J13-Pad1): track 0.00 -> 30.5 mm
- net Net-(D2-Pad2): track 0.00 -> 25.4 mm
- net Net-(J12-Pad1): track 0.00 -> 22.9 mm
- net Net-(J10-Pad1): track 0.00 -> 22.7 mm
- net Net-(D3-Pad2): track 0.00 -> 10.2 mm
- net Net-(D3-Pad1): track 0.00 -> 10.2 mm
- net Net-(D2-Pad1): track 0.00 -> 10.2 mm
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
Commit message: make arduino part of pcb
Parts:
- added J33: switch_TIMER, Connector_Wire:SolderWirePad_1x01_Drill0.8mm, F.Cu at (105.4, -87.4)
- added J34: switch_LIGHT, Connector_Wire:SolderWirePad_1x01_Drill0.8mm, F.Cu at (127.0, -95.2)
- added J35: switch_GND, Connector_Wire:SolderWirePad_1x01_Drill0.8mm, F.Cu at (127.5, -87.4)
- added J36: switch_TIMER, Connector_Wire:SolderWirePad_1x01_Drill0.8mm, F.Cu at (45.7, 116.8)
- added J37: switch_LIGHT, Connector_Wire:SolderWirePad_1x01_Drill0.8mm, F.Cu at (45.7, 121.9)
- added J38: switch_GND, Connector_Wire:SolderWirePad_1x01_Drill0.8mm, F.Cu at (45.7, 127.0)
- added SW5: MODE, ToggleSwitch:SW_Toggle_Blue_wSlots, F.Cu at (91.4, -101.6)
- moved J1 168.0 mm to (121.9, 88.9)
- moved SW1 165.4 mm to (228.6, 132.1)
- moved SW2 165.4 mm to (246.4, 132.1)
- moved SW3 165.4 mm to (264.2, 132.1)
- moved SW4 165.4 mm to (210.8, 132.1)
- moved D1 165.4 mm to (170.2, 114.3)
- moved D2 165.4 mm to (170.2, 124.5)
- moved D3 165.4 mm to (170.2, 134.6)
- moved J10 165.4 mm to (210.8, 147.3)
- moved J11 165.4 mm to (195.6, 147.3)
- moved J12 165.4 mm to (129.5, 147.3)
- moved J13 165.4 mm to (124.5, 147.3)
- moved J14 165.4 mm to (180.3, 147.3)
- moved J15 165.4 mm to (185.4, 147.3)
- moved J3 165.4 mm to (160.0, 147.3)
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Routing:
- net GND: track 0.00 -> 406.4 mm, vias 0 -> 7
- net +5V: track 0.00 -> 228.6 mm, vias 0 -> 3
- net Net-(A1-Pad20): track 0.00 -> 101.6 mm, vias 0 -> 4
- net Net-(A1-Pad15): track 0.00 -> 55.9 mm
- net Net-(A1-Pad14): track 0.00 -> 53.3 mm
- net Net-(A1-Pad5): track 0.00 -> 48.3 mm
- net Net-(A1-Pad6): track 0.00 -> 45.7 mm
- net Net-(A1-Pad13): track 0.00 -> 45.7 mm, vias 0 -> 2
- net Net-(A1-Pad7): track 0.00 -> 43.2 mm
- net Net-(A1-Pad12): track 0.00 -> 40.6 mm
- net Net-(A1-Pad11): track 0.00 -> 38.1 mm
- net Net-(A1-Pad8): track 0.00 -> 33.0 mm
- net Net-(A1-Pad9): track 0.00 -> 30.5 mm
- net Net-(J2-Pad1): track 0.00 -> 27.9 mm, vias 0 -> 2
- net Net-(A1-Pad10): track 0.00 -> 27.9 mm
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
Commit message: update schematic to KiCad 6
Parts:
- removed J33: switch_TIMER, Connector_Wire:SolderWirePad_1x01_Drill0.8mm
- removed J34: switch_LIGHT, Connector_Wire:SolderWirePad_1x01_Drill0.8mm
- removed J35: switch_GND, Connector_Wire:SolderWirePad_1x01_Drill0.8mm
- removed SW5: MODE, ToggleSwitch:SW_Toggle_Blue_wSlots
- J1: value lamp VCC -> lamp VCC (out)
- J2: value lamp GND -> lamp GND (out)
- J30: value VCC amp -> VCC lamp (in)
- J31: value GND lamp -> GND lamp (in)
- moved J1 152.0 mm to (271.8, 114.3)
- moved J31 151.2 mm to (271.8, 96.5)
- moved J2 150.9 mm to (271.8, 99.1)
- moved J30 150.4 mm to (271.8, 106.7)
- moved A1 148.4 mm to (218.4, 73.7)
- moved J16 148.4 mm to (193.0, 61.0)
- moved J17 148.4 mm to (193.0, 66.0)
- moved J18 148.4 mm to (193.0, 71.1)
- moved J19 148.4 mm to (193.0, 76.2)
- moved J20 148.4 mm to (193.0, 99.1)
- moved J21 148.4 mm to (193.0, 83.8)
- moved J22 148.4 mm to (193.0, 88.9)
- moved J23 148.4 mm to (193.0, 94.0)
- moved J24 148.4 mm to (193.0, 104.1)
- moved J25 148.4 mm to (193.0, 111.8)
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Connections:
- A1 pad 1: Net-(A1-Pad1) -> unconnected-(A1-Pad1)
- A1 pad 16: Net-(A1-Pad16) -> unconnected-(A1-Pad16)
- A1 pad 17: Net-(A1-Pad17) -> unconnected-(A1-Pad17)
- A1 pad 18: Net-(A1-Pad18) -> unconnected-(A1-Pad18)
- A1 pad 19: Net-(A1-Pad19) -> unconnected-(A1-Pad19)
- A1 pad 2: Net-(A1-Pad2) -> unconnected-(A1-Pad2)
- A1 pad 21: Net-(A1-Pad21) -> unconnected-(A1-Pad21)
- A1 pad 22: Net-(A1-Pad22) -> unconnected-(A1-Pad22)
- A1 pad 25: Net-(A1-Pad25) -> unconnected-(A1-Pad25)
- A1 pad 26: Net-(A1-Pad26) -> unconnected-(A1-Pad26)
- A1 pad 27: Net-(A1-Pad27) -> unconnected-(A1-Pad27)
- A1 pad 28: Net-(A1-Pad28) -> unconnected-(A1-Pad28)
- A1 pad 3: Net-(A1-Pad3) -> unconnected-(A1-Pad3)
Routing:
- net GND: track 406.4 -> 292.1 mm, vias 7 -> 5
- net Net-(D3-Pad2): track 10.2 -> 58.4 mm
- net Net-(D2-Pad2): track 25.4 -> 66.0 mm
- net Net-(J7-Pad1): track 60.8 -> 25.3 mm
- net Net-(J14-Pad1): track 58.4 -> 22.9 mm, vias 2 -> 0
- net Net-(J15-Pad1): track 66.0 -> 30.5 mm, vias 2 -> 0
- net Net-(D1-Pad2): track 40.6 -> 73.7 mm
- net Net-(J6-Pad1): track 33.0 -> 66.0 mm
- net Net-(J10-Pad1): track 22.7 -> 50.8 mm
- net Net-(A1-Pad13): track 45.7 -> 17.8 mm, vias 2 -> 0
- net Net-(Q1-Pad1): track 15.2 -> 40.6 mm
- net Net-(J8-Pad1): track 48.1 -> 25.3 mm
- net Net-(J13-Pad1): track 30.5 -> 50.8 mm
- net Net-(J12-Pad1): track 22.9 -> 43.2 mm
- net Net-(A1-Pad20): track 101.6 -> 91.4 mm, vias 4 -> 2
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Other:
- net class Default removed
