File: schematic/schematic.sch (KiCad schematic (older format))
At the start: 15 parts, among them Q1 IRLZ34N, SW1 MODE, SW2 UP, SW3 DOWN, SW4 SW_Push, U1 TM1637Display

Commit message: draw schematics
Parts:
- removed R2, R3, R4: R, Resistor_THT:R_Axial_DIN0204_L3.6mm_D1.6mm_P5.08mm_Vertical, symbol Device:R
- removed SW4: SW_Push, Button_Switch_THT:SW_PUSH_6mm_H5mm, symbol Switch:SW_Push
- added R? (x4): R, Resistor_THT:R_Axial_DIN0204_L3.6mm_D1.6mm_P5.08mm_Vertical, symbol Device:R
- added SW?: MODE, Button_Switch_THT:SW_PUSH_6mm_H5mm, symbol Switch:SW_Push
- SW1: value MODE -> UP
- SW2: value UP -> DOWN
- SW3: value DOWN -> CONFIRM
Connections:
- net labels added: +5V, GND, display_clk, display_dio, display_gnd, display_vcc, lamp_gnd, lamp_vcc, led_off, led_on, led_time, leds_gnd, switch_confirm, switch_down, switch_mode, switch_up, switchs_gnd
- wire segments 6 -> 110
Other:
- moved on the sheet: A1, D1, D2, D3, Q1, R1, RTC1, SW1, SW2, SW3, U1

Commit message: update board
Parts:
- added J1: lamp VCC, Connector_Wire:SolderWirePad_1x01_Drill0.8mm, symbol Connector_Generic:Conn_01x01
- added J10, J23: button MODE, Connector_Wire:SolderWirePad_1x01_Drill0.8mm, symbol Connector_Generic:Conn_01x01
- added J11, J24: button GND, Connector_Wire:SolderWirePad_1x01_Drill0.8mm, symbol Connector_Generic:Conn_01x01
- added J12, J25: display DIO, Connector_Wire:SolderWirePad_1x01_Drill0.8mm, symbol Connector_Generic:Conn_01x01
- added J13, J26: display CLK, Connector_Wire:SolderWirePad_1x01_Drill0.8mm, symbol Connector_Generic:Conn_01x01
- added J14, J27: display VCC, Connector_Wire:SolderWirePad_1x01_Drill0.8mm, symbol Connector_Generic:Conn_01x01
- added J15, J28: display GND, Connector_Wire:SolderWirePad_1x01_Drill0.8mm, symbol Connector_Generic:Conn_01x01
- added J16, J3: led OFF, Connector_Wire:SolderWirePad_1x01_Drill0.8mm, symbol Connector_Generic:Conn_01x01
- added J17, J4: led ON, Connector_Wire:SolderWirePad_1x01_Drill0.8mm, symbol Connector_Generic:Conn_01x01
- added J18, J5: led TIME, Connector_Wire:SolderWirePad_1x01_Drill0.8mm, symbol Connector_Generic:Conn_01x01
- added J19, J6: led GND, Connector_Wire:SolderWirePad_1x01_Drill0.8mm, symbol Connector_Generic:Conn_01x01
- added J2: lamp GND, Connector_Wire:SolderWirePad_1x01_Drill0.8mm, symbol Connector_Generic:Conn_01x01
- added J20, J7: button CONFIRM, Connector_Wire:SolderWirePad_1x01_Drill0.8mm, symbol Connector_Generic:Conn_01x01
- added J21, J8: button DOWN, Connector_Wire:SolderWirePad_1x01_Drill0.8mm, symbol Connector_Generic:Conn_01x01
- added J22, J9: button UP, Connector_Wire:SolderWirePad_1x01_Drill0.8mm, symbol Connector_Generic:Conn_01x01
- added J29: VCC, Connector_Wire:SolderWirePad_1x01_Drill0.8mm, symbol Connector_Generic:Conn_01x01
- added J30: VCC amp, Connector_Wire:SolderWirePad_1x01_Drill0.8mm, symbol Connector_Generic:Conn_01x01
- added J31: GND lamp, Connector_Wire:SolderWirePad_1x01_Drill0.8mm, symbol Connector_Generic:Conn_01x01
- added J32: GND, Connector_Wire:SolderWirePad_1x01_Drill0.8mm, symbol Connector_Generic:Conn_01x01
- R1: footprint Resistor_THT:R_Axial_DIN0204_L3.6mm_D1.6mm_P5.08mm_Vertical -> Resistor_THT:R_Axial_DIN0207_L6.3mm_D2.5mm_P10.16mm_Horizontal
- R2, R3, R4, R5: renamed from R?; footprint Resistor_THT:R_Axial_DIN0204_L3.6mm_D1.6mm_P5.08mm_Vertical -> Resistor_THT:R_Axial_DIN0207_L6.3mm_D2.5mm_P10.16mm_Horizontal
- SW1, SW2, SW3: footprint Button_Switch_THT:SW_PUSH_6mm_H5mm -> Button_Switch_THT:SW_PUSH-12mm
- SW4: renamed from SW?; footprint Button_Switch_THT:SW_PUSH_6mm_H5mm -> Button_Switch_THT:SW_PUSH-12mm
Connections:
- net +5V: now also J27.1 (Pin_1), J29.1 (Pin_1); no longer U1.4 (5V)
- net GND: now also J19.1 (Pin_1), J24.1 (Pin_1), J28.1 (Pin_1), J32.1 (Pin_1); no longer Q1.3 (S), R2.2, R3.2, R4.2, SW1.1, SW2.1, SW3.1, SW4.1, U1.3 (GND)
- net display_clk: no longer names the net of A1.12 (D9)
- net display_clk: now also J26.1 (Pin_1); no longer U1.1 (CLK)
- net display_dio: no longer names the net of A1.11 (D8)
- net display_dio: now also J25.1 (Pin_1); no longer U1.2 (DIO)
- net lamp_gnd: no longer names the net of Q1.2 (D)
- net lamp_gnd: now also J2.1 (Pin_1)
- net led_off: no longer names the net of A1.5 (D2)
- net led_off: now also J16.1 (Pin_1); no longer D1.2 (A)
- net led_on: no longer names the net of A1.6 (D3)
- net led_on: now also J17.1 (Pin_1); no longer D2.2 (A)
- net led_time: no longer names the net of A1.7 (D4)
- net led_time: now also J18.1 (Pin_1); no longer D3.2 (A)
- net switch_confirm: no longer names the net of A1.20 (A1)
- net switch_confirm: now also J20.1 (Pin_1); no longer SW3.2
- net switch_down: no longer names the net of A1.8 (D5)
- net switch_down: now also J21.1 (Pin_1); no longer SW2.2
- net switch_mode: no longer names the net of A1.10 (D7)
- net switch_mode: now also J23.1 (Pin_1); no longer SW4.2
- net switch_up: no longer names the net of A1.9 (D6)
- net switch_up: now also J22.1 (Pin_1); no longer SW1.2
- new net: J13.1 (Pin_1), U1.1 (CLK)
- new net: J12.1 (Pin_1), U1.2 (DIO)
- new net: J15.1 (Pin_1), U1.3 (GND)
- new net: J14.1 (Pin_1), U1.4 (5V)
- new net: J11.1 (Pin_1), SW1.1, SW2.1, SW3.1, SW4.1
- new net: J7.1 (Pin_1), SW3.2
- new net: J9.1 (Pin_1), SW1.2
- new net: J31.1 (Pin_1), Q1.3 (S)
- new net: D1.2 (A), J3.1 (Pin_1)
- new net: D2.2 (A), J4.1 (Pin_1)
- new net: D3.2 (A), J5.1 (Pin_1)
- new net: J8.1 (Pin_1), SW2.2
- new net: J1.1 (Pin_1), J30.1 (Pin_1)
- new net: J6.1 (Pin_1), R2.2, R3.2, R4.2
- new net: J10.1 (Pin_1), SW4.2

Commit message: make arduino part of pcb
Parts:
- added J33, J36: switch_TIMER, Connector_Wire:SolderWirePad_1x01_Drill0.8mm, symbol Connector_Generic:Conn_01x01
- added J34, J37: switch_LIGHT, Connector_Wire:SolderWirePad_1x01_Drill0.8mm, symbol Connector_Generic:Conn_01x01
- added J35, J38: switch_GND, Connector_Wire:SolderWirePad_1x01_Drill0.8mm, symbol Connector_Generic:Conn_01x01
- added SW5: MODE, symbol Switch:SW_SPDT_MSM
Connections:
- net GND: now also J38.1 (Pin_1)
- net at A1.14 (D11): now also J36.1 (Pin_1)
- net at A1.15 (D12): now also J37.1 (Pin_1)
- new net: J33.1 (Pin_1), SW5.1
- new net: J35.1 (Pin_1), SW5.2
- new net: J34.1 (Pin_1), SW5.3
Other:
- moved on the sheet: A1, D1, D2, D3, Q1, R1, R2, R3, R4, R5, RTC1, SW1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

Commit message: update schematic to KiCad 6
Parts:
- SW5: footprint (none) -> ToggleSwitch:SW_Toggle_Blue_wSlots
Changed lines of the file:
@@
 F 0 "SW5" H 3500 5535 50  0000 C CNN
 F 1 "MODE" H 3500 5444 50  0000 C CNN
-F 2 "" H 3500 5250 50  0001 C CNN
+F 2 "ToggleSwitch:SW_Toggle_Blue_wSlots" H 3500 5250 50  0001 C CNN
 F 3 "~" H 3500 5250 50  0001 C CNN
 	1    3500 5250
